Commit message: 24/9-15:26

File: ur_description/urdf/eef.xacro (robot description, xacro)
@@ -1,17 +1,75 @@
 <?xml version="1.0"?>
 <robot xmlns:xacro="http://wiki.ros.org/xacro" name="robotiq_gripper">
-    <xacro:include filename="$(find ur_description)/urdf/robotiq_2f_85_macro.urdf.xacro" />
+    <!--xacro:include filename="$(find ur_description)/urdf/robotiq_2f_85_macro.urdf.xacro" />
     <xacro:robotiq_gripper name="RobotiqGripperHardwareInterface" prefix="" parent="tool0" >
         <origin xyz="0 0 0" rpy="0 0 0" />
-    </xacro:robotiq_gripper>
+    </xacro:robotiq_gripper-->
+    <xacro:include filename="$(find robotiq_description)/urdf/robotiq_85_gripper.urdf.xacro" />
+    <link name="robotiq_coupler">
+        <visual>
+            <geometry>
+                <mesh filename="package://ur_description/meshes/robotiq_85_coupler.stl" />
+                <origin xyz="0 0 0" rpy="0 0 0" />
+            </geometry>
+            <material name="flat_black"/>
+        </visual>
+        <collision>
+            <geometry>
+                <mesh filename="package://ur_description/meshes/robotiq_85_coupler.stl" />
+                <origin xyz="0 0 0" rpy="0 0 0" />
+            </geometry>
+        </collision>
+        <inertial>
+            <origin xyz="0 0 0" rpy="0 0 0" />
+            <mass value="0.168" />
+            <inertia ixx="6.69695624e-05" ixy="5.21511788e-09" ixz="-2.74383009e-08"
+                    iyy="7.85088161e-05" iyz="5.41105193e-07" izz="1.41819717e-04"/>
+        </inertial>
+    </link>
+    <gazebo reference="robotiq_coupler">
+        <mu1>0.2</mu1>
+        <mu2>0.2</mu2>
+        <material>Gazebo/Red</material>
+    </gazebo>
+    <joint name="robotiq_coupler_joint" type="fixed">
+        <origin xyz="0 0 0" rpy="0 0 0" />
+        <parent link="tool0"/>
+        <child link="robotiq_coupler"/>
+    </joint>
+    <!-- Attach the robotiq 85 gripper -->
+    <xacro:robotiq_85_gripper prefix="" parent="tool0" >
+        <origin xyz="0 0 0.007" rpy="0 ${-pi/2} ${pi}"/>
+    </xacro:robotiq_85_gripper>
+    <!-- Equivalent to the OpenRAVE manipulator denso_robotiq_85_gripper -->
+    <link name="ee_link" />
+    <joint name="manipulator_dummy_joint" type="fixed">
+        <origin xyz="0 0 0.17" rpy="0 0 0" />
+        <parent link="tool0"/>
+        <child link="ee_link"/>
+    </joint>
+    <!-- Gazebo FT sensor plugin -->
+    <!--gazebo reference="wrist_3_joint">
+        <provideFeedback>true</provideFeedback>
+    </gazebo>
+    <gazebo>
+        <plugin name="ft_sensor_plugin" filename="libgazebo_ros_ft_sensor.so">
+        <updateRate>250.0</updateRate>
+        <topicName>ft_sensor/raw</topicName>
+        <gaussianNoise>0.0</gaussianNoise>
+        <jointName>wrist_3_joint</jointName>
+        </plugin>
+    </gazebo-->
+    <!-- Gazebo grasping plugin -->
+    <gazebo>
+        <gripper name="gazebo_gripper">
+        <grasp_check>
+            <attach_steps>2</attach_steps>
+            <detach_steps>2</detach_steps>
+            <min_contact_count>3</min_contact_count>
+        </grasp_check>
+        <gripper_link>robotiq_85_left_finger_tip_link</gripper_link>
+        <gripper_link>robotiq_85_right_finger_tip_link</gripper_link>
+        <palm_link>robotiq_85_base_link</palm_link>
+        </gripper>
+    </gazebo>
 </robot>
-<!--robot name="robotiq_85_gripper" xmlns:xacro="http://ros.org/wiki/xacro">
-    <xacro:include filename="$(find ur_description)/urdf/robotiq_85_gripper.urdf.xacro" />
-    <gazebo>
-        <plugin name="gazebo_ros_control" filename="libgazebo_ros_control.so">
-            <robotNamespace>/robotiq_gripper</robotNamespace>
-        </plugin>
-    </gazebo>
-    <xacro:robotiq_85_gripper prefix="" parent="tool0" origin_xyz="0 0 0" origin_rpy="0 0 0" >
-    </xacro:robotiq_85_gripper>
-</robot-->

File: ur_description/urdf/robotiq_2f_85_macro.urdf.xacro (robot description, xacro)
@@ -259,5 +259,5 @@
             <axis xyz="0 -1 0" />
             <origin xyz="-0.0127 0.0 0.06142" rpy="0 0 0" />
-            <mimic joint="${prefix}robotiq_85_left_knuckle_joint" multiplier="-1" />
+            <!--mimic joint="${prefix}robotiq_85_left_knuckle_joint" multiplier="-1" /-->
         </joint>
         <joint name="${prefix}robotiq_85_left_finger_tip_joint" type="continuous">
@@ -266,5 +266,5 @@
             <axis xyz="0 -1 0" />
             <origin xyz="0.00563134 0.0 0.04718515" rpy="0 0 0" />
-            <mimic joint="${prefix}robotiq_85_left_knuckle_joint" multiplier="-1" />
+            <!--mimic joint="${prefix}robotiq_85_left_knuckle_joint" multiplier="-1" /-->
         </joint>
         <joint name="${prefix}robotiq_85_right_finger_tip_joint" type="continuous">
@@ -275,4 +275,16 @@
             <mimic joint="${prefix}robotiq_85_left_knuckle_joint" />
         </joint>
+        <!--joint name="${prefix}robotiq_85_left_inner_knuckle_tip_joint" type="continuous">
+            <parent link="${prefix}robotiq_85_left_finger_tip_link" />
+            <child link="${prefix}robotiq_85_left_inner_knuckle_link" />
+            <axis xyz="0 -1 0" />
+            <origin xyz="0 0 0" rpy="0 0 0" />
+        </joint>
+        <joint name="${prefix}robotiq_85_right_inner_knuckle_tip_joint" type="continuous">
+            <parent link="${prefix}robotiq_85_right_finger_tip_link" />
+            <child link="${prefix}robotiq_85_right_inner_knuckle_link" />
+            <axis xyz="0 -1 0" />
+            <origin xyz="0 0 0" rpy="0 0 0" />
+        </joint-->
     </xacro:macro>
 </robot>

File: ur_description/urdf/ur_macro.xacro (robot description, xacro)
@@ -363,7 +363,7 @@
     </joint>
     <!-- ROS-Industrial 'flange' frame - attachment point for EEF models -->
-    <link name="${tf_prefix}flange" />
+    <link name="${tf_prefix}flange"/>
     <joint name="${tf_prefix}wrist_3-flange" type="fixed">
-      <parent link="${tf_prefix}wrist_3_link" />
+      <parent link="${tf_prefix}wrist_3_link"/>
       <child link="${tf_prefix}flange" />
       <origin xyz="0 0 0" rpy="0 ${-pi/2.0} ${-pi/2.0}" />
@@ -373,15 +373,9 @@
     <joint name="${tf_prefix}flange-tool0" type="fixed">
       <!-- default toolframe - X+ left, Y+ up, Z+ front -->
-      <origin xyz="0 0 0" rpy="${pi/2.0} 0 ${pi/2.0}"/>
+      <origin xyz="0 0 0.001" rpy="${pi/2.0} 0 ${pi/2.0}"/>
       <parent link="${tf_prefix}flange"/>
       <child link="${tf_prefix}tool0"/>
     </joint>
-    <!-- Bao gồm gripper -->
-    <xacro:include filename="$(find ur_description)/urdf/eef.xacro" />
-    <!--joint name="tool0-gripper" type="fixed">
-      <origin xyz="0 0 0" rpy="0 0 0"/>
-      <parent link="${tf_prefix}tool0"/>
-      <child link="world"/>
-    </joint-->
+    <!--xacro:include filename="$(find ur_description)/urdf/eefold.xacro" /-->
   </xacro:macro>
 </robot>

File: ur_moveit_config/srdf/ur_macro.srdf.xacro (robot description, xacro)
@@ -12,5 +12,6 @@
     <!--SUBGROUPS - Groups can also be formed by referencing to already defined group names-->
     <group name="${prefix}${name}_manipulator">
-      <chain base_link="${prefix}base_link" tip_link="${prefix}tool0" />
+      <chain base_link="${prefix}base_link" tip_link="${prefix}tool0"/>
+      <!--chain base_link="${prefix}base_link" tip_link="ee_link"  /-->
     </group>
     <!--GROUP STATES - Purpose - Define a named state for a particular group, in terms of joint values. This is useful to define states like 'folded arms'-->
@@ -53,4 +54,99 @@
     <disable_collisions link1="${prefix}wrist_1_link" link2="${prefix}wrist_3_link" reason="Never" />
     <disable_collisions link1="${prefix}wrist_2_link" link2="${prefix}wrist_3_link" reason="Adjacent" />
+    <!--disable_collisions link1="${prefix}base_link" link2="${prefix}shoulder_link" reason="Adjacent" />
+    <disable_collisions link1="${prefix}tool0" link2="robotiq_85_base_link" reason="Never" />
+    <disable_collisions link1="${prefix}tool0" link2="robotiq_85_left_finger_link" reason="Never" />
+    <disable_collisions link1="${prefix}tool0" link2="robotiq_85_left_finger_tip_link" reason="Never" />
+    <disable_collisions link1="${prefix}tool0" link2="robotiq_85_left_inner_knuckle_link" reason="Never" />
+    <disable_collisions link1="${prefix}tool0" link2="robotiq_85_left_knuckle_link" reason="Never" />
+    <disable_collisions link1="${prefix}tool0" link2="robotiq_85_right_finger_link" reason="Never" />
+    <disable_collisions link1="${prefix}tool0" link2="robotiq_85_right_finger_tip_link" reason="Never" />
+    <disable_collisions link1="${prefix}tool0" link2="robotiq_85_right_inner_knuckle_link" reason="Never" />
+    <disable_collisions link1="${prefix}tool0" link2="robotiq_85_right_knuckle_link" reason="Never" />
+    <disable_collisions link1="${prefix}tool0" link2="robotiq_coupler" reason="Never" />
+    <disable_collisions link1="${prefix}tool0" link2="${prefix}wrist_1_link" reason="Never" />
+    <disable_collisions link1="${prefix}tool0" link2="${prefix}wrist_2_link" reason="Never" />
+    <disable_collisions link1="${prefix}tool0" link2="${prefix}wrist_3_link" reason="Adjacent" />
+    <disable_collisions link1="${prefix}forearm_link" link2="${prefix}upper_arm_link" reason="Adjacent" />
+    <disable_collisions link1="${prefix}forearm_link" link2="${prefix}wrist_1_link" reason="Adjacent" />
+    <disable_collisions link1="robotiq_85_base_link" link2="robotiq_85_left_finger_link" reason="Never" />
+    <disable_collisions link1="robotiq_85_base_link" link2="robotiq_85_left_finger_tip_link" reason="Never" />
+    <disable_collisions link1="robotiq_85_base_link" link2="robotiq_85_left_inner_knuckle_link" reason="Adjacent" />
+    <disable_collisions link1="robotiq_85_base_link" link2="robotiq_85_left_knuckle_link" reason="Adjacent" />
+    <disable_collisions link1="robotiq_85_base_link" link2="robotiq_85_right_finger_link" reason="Never" />
+    <disable_collisions link1="robotiq_85_base_link" link2="robotiq_85_right_finger_tip_link" reason="Never" />
+    <disable_collisions link1="robotiq_85_base_link" link2="robotiq_85_right_inner_knuckle_link" reason="Adjacent" />
+    <disable_collisions link1="robotiq_85_base_link" link2="robotiq_85_right_knuckle_link" reason="Adjacent" />
+    <disable_collisions link1="robotiq_85_base_link" link2="robotiq_coupler" reason="Adjacent" />
+    <disable_collisions link1="robotiq_85_base_link" link2="${prefix}wrist_1_link" reason="Never" />
+    <disable_collisions link1="robotiq_85_base_link" link2="${prefix}wrist_2_link" reason="Never" />
+    <disable_collisions link1="robotiq_85_base_link" link2="${prefix}wrist_3_link" reason="Never" />
+    <disable_collisions link1="robotiq_85_left_finger_link" link2="robotiq_85_left_finger_tip_link" reason="Default" />
+    <disable_collisions link1="robotiq_85_left_finger_link" link2="robotiq_85_left_inner_knuckle_link" reason="Never" />
+    <disable_collisions link1="robotiq_85_left_finger_link" link2="robotiq_85_left_knuckle_link" reason="Adjacent" />
+    <disable_collisions link1="robotiq_85_left_finger_link" link2="robotiq_85_right_finger_link" reason="Never" />
+    <disable_collisions link1="robotiq_85_left_finger_link" link2="robotiq_85_right_finger_tip_link" reason="Never" />
+    <disable_collisions link1="robotiq_85_left_finger_link" link2="robotiq_85_right_inner_knuckle_link" reason="Never" />
+    <disable_collisions link1="robotiq_85_left_finger_link" link2="robotiq_85_right_knuckle_link" reason="Never" />
+    <disable_collisions link1="robotiq_85_left_finger_link" link2="robotiq_coupler" reason="Never" />
+    <disable_collisions link1="robotiq_85_left_finger_link" link2="${prefix}wrist_1_link" reason="Never" />
+    <disable_collisions link1="robotiq_85_left_finger_link" link2="${prefix}wrist_2_link" reason="Never" />
+    <disable_collisions link1="robotiq_85_left_finger_link" link2="${prefix}wrist_3_link" reason="Never" />
+    <disable_collisions link1="robotiq_85_left_finger_tip_link" link2="robotiq_85_left_inner_knuckle_link" reason="Adjacent" />
+    <disable_collisions link1="robotiq_85_left_finger_tip_link" link2="robotiq_85_left_knuckle_link" reason="Never" />
+    <disable_collisions link1="robotiq_85_left_finger_tip_link" link2="robotiq_85_right_finger_link" reason="Never" />
+    <disable_collisions link1="robotiq_85_left_finger_tip_link" link2="robotiq_85_right_finger_tip_link" reason="Never" />
+    <disable_collisions link1="robotiq_85_left_finger_tip_link" link2="robotiq_85_right_inner_knuckle_link" reason="Never" />
+    <disable_collisions link1="robotiq_85_left_finger_tip_link" link2="robotiq_85_right_knuckle_link" reason="Never" />
+    <disable_collisions link1="robotiq_85_left_finger_tip_link" link2="robotiq_coupler" reason="Never" />
+    <disable_collisions link1="robotiq_85_left_finger_tip_link" link2="${prefix}wrist_1_link" reason="Never" />
+    <disable_collisions link1="robotiq_85_left_finger_tip_link" link2="${prefix}wrist_2_link" reason="Never" />
+    <disable_collisions link1="robotiq_85_left_finger_tip_link" link2="${prefix}wrist_3_link" reason="Never" />
+    <disable_collisions link1="robotiq_85_left_inner_knuckle_link" link2="robotiq_85_left_knuckle_link" reason="Never" />
+    <disable_collisions link1="robotiq_85_left_inner_knuckle_link" link2="robotiq_85_right_finger_link" reason="Never" />
+    <disable_collisions link1="robotiq_85_left_inner_knuckle_link" link2="robotiq_85_right_finger_tip_link" reason="Never" />
+    <disable_collisions link1="robotiq_85_left_inner_knuckle_link" link2="robotiq_85_right_inner_knuckle_link" reason="Never" />
+    <disable_collisions link1="robotiq_85_left_inner_knuckle_link" link2="robotiq_85_right_knuckle_link" reason="Never" />
+    <disable_collisions link1="robotiq_85_left_inner_knuckle_link" link2="robotiq_coupler" reason="Never" />
+    <disable_collisions link1="robotiq_85_left_inner_knuckle_link" link2="${prefix}wrist_1_link" reason="Never" />
+    <disable_collisions link1="robotiq_85_left_inner_knuckle_link" link2="${prefix}wrist_2_link" reason="Never" />
+    <disable_collisions link1="robotiq_85_left_inner_knuckle_link" link2="${prefix}wrist_3_link" reason="Never" />
+    <disable_collisions link1="robotiq_85_left_knuckle_link" link2="robotiq_85_right_finger_link" reason="Never" />
+    <disable_collisions link1="robotiq_85_left_knuckle_link" link2="robotiq_85_right_finger_tip_link" reason="Never" />
+    <disable_collisions link1="robotiq_85_left_knuckle_link" link2="robotiq_85_right_inner_knuckle_link" reason="Never" />
+    <disable_collisions link1="robotiq_85_left_knuckle_link" link2="robotiq_85_right_knuckle_link" reason="Never" />
+    <disable_collisions link1="robotiq_85_left_knuckle_link" link2="robotiq_coupler" reason="Never" />
+    <disable_collisions link1="robotiq_85_left_knuckle_link" link2="${prefix}wrist_1_link" reason="Never" />
+    <disable_collisions link1="robotiq_85_left_knuckle_link" link2="${prefix}wrist_2_link" reason="Never" />
+    <disable_collisions link1="robotiq_85_left_knuckle_link" link2="${prefix}wrist_3_link" reason="Never" />
+    <disable_collisions link1="robotiq_85_right_finger_link" link2="robotiq_85_right_finger_tip_link" reason="Default" />
+    <disable_collisions link1="robotiq_85_right_finger_link" link2="robotiq_85_right_inner_knuckle_link" reason="Never" />
+    <disable_collisions link1="robotiq_85_right_finger_link" link2="robotiq_85_right_knuckle_link" reason="Adjacent" />
+    <disable_collisions link1="robotiq_85_right_finger_link" link2="robotiq_coupler" reason="Never" />
+    <disable_collisions link1="robotiq_85_right_finger_link" link2="${prefix}wrist_1_link" reason="Never" />
+    <disable_collisions link1="robotiq_85_right_finger_link" link2="${prefix}wrist_2_link" reason="Never" />
+    <disable_collisions link1="robotiq_85_right_finger_link" link2="${prefix}wrist_3_link" reason="Never" />
+    <disable_collisions link1="robotiq_85_right_finger_tip_link" link2="robotiq_85_right_inner_knuckle_link" reason="Adjacent" />
+    <disable_collisions link1="robotiq_85_right_finger_tip_link" link2="robotiq_85_right_knuckle_link" reason="Never" />
+    <disable_collisions link1="robotiq_85_right_finger_tip_link" link2="robotiq_coupler" reason="Never" />
+    <disable_collisions link1="robotiq_85_right_finger_tip_link" link2="${prefix}wrist_1_link" reason="Never" />
+    <disable_collisions link1="robotiq_85_right_finger_tip_link" link2="${prefix}wrist_2_link" reason="Never" />
+    <disable_collisions link1="robotiq_85_right_finger_tip_link" link2="${prefix}wrist_3_link" reason="Never" />
+    <disable_collisions link1="robotiq_85_right_inner_knuckle_link" link2="robotiq_85_right_knuckle_link" reason="Never" />
+    <disable_collisions link1="robotiq_85_right_inner_knuckle_link" link2="robotiq_coupler" reason="Never" />
+    <disable_collisions link1="robotiq_85_right_inner_knuckle_link" link2="${prefix}wrist_1_link" reason="Never" />
+    <disable_collisions link1="robotiq_85_right_inner_knuckle_link" link2="${prefix}wrist_2_link" reason="Never" />
+    <disable_collisions link1="robotiq_85_right_inner_knuckle_link" link2="${prefix}wrist_3_link" reason="Never" />
+    <disable_collisions link1="robotiq_85_right_knuckle_link" link2="robotiq_coupler" reason="Never" />
+    <disable_collisions link1="robotiq_85_right_knuckle_link" link2="${prefix}wrist_1_link" reason="Never" />
+    <disable_collisions link1="robotiq_85_right_knuckle_link" link2="${prefix}wrist_2_link" reason="Never" />
+    <disable_collisions link1="robotiq_85_right_knuckle_link" link2="${prefix}wrist_3_link" reason="Never" />
+    <disable_collisions link1="robotiq_coupler" link2="${prefix}wrist_1_link" reason="Never" />
+    <disable_collisions link1="robotiq_coupler" link2="${prefix}wrist_2_link" reason="Never" />
+    <disable_collisions link1="robotiq_coupler" link2="${prefix}wrist_3_link" reason="Adjacent" />
+    <disable_collisions link1="${prefix}shoulder_link" link2="${prefix}upper_arm_link" reason="Adjacent" />
+    <disable_collisions link1="${prefix}wrist_1_link" link2="${prefix}wrist_2_link" reason="Adjacent" />
+    <disable_collisions link1="${prefix}wrist_1_link" link2="${prefix}wrist_3_link" reason="Never" />
+    <disable_collisions link1="${prefix}wrist_2_link" link2="${prefix}wrist_3_link" reason="Adjacent" /-->
   </xacro:macro>
 </robot>
