Commit message: 36/9-15:48

File: robotiq_description/urdf/robotiq_85_gripper.transmission.xacro (robot description, xacro)
@@ -16,17 +16,17 @@
     <!-- Mimic joints -->
     <gazebo>
-      <plugin filename="libgazebo_mimic_joint_plugin.so" name="${prefix}mimic_robotiq_85_1">
+      <plugin filename="libroboticsgroup_gazebo_mimic_joint_plugin.so" name="${prefix}mimic_robotiq_85_1">
         <joint>${prefix}robotiq_85_left_knuckle_joint</joint>
         <mimicJoint>${prefix}robotiq_85_right_knuckle_joint</mimicJoint>
       </plugin>
-      <plugin filename="libgazebo_mimic_joint_plugin.so" name="${prefix}mimic_robotiq_85_2">
+      <plugin filename="libroboticsgroup_gazebo_mimic_joint_plugin.so" name="${prefix}mimic_robotiq_85_2">
         <joint>${prefix}robotiq_85_left_knuckle_joint</joint>
         <mimicJoint>${prefix}robotiq_85_left_inner_knuckle_joint</mimicJoint>
       </plugin>
-      <plugin filename="libgazebo_mimic_joint_plugin.so" name="${prefix}mimic_robotiq_85_3">
+      <plugin filename="libroboticsgroup_gazebo_mimic_joint_plugin.so" name="${prefix}mimic_robotiq_85_3">
         <joint>${prefix}robotiq_85_left_knuckle_joint</joint>
         <mimicJoint>${prefix}robotiq_85_right_inner_knuckle_joint</mimicJoint>
       </plugin>
-      <plugin filename="libgazebo_mimic_joint_plugin.so" name="${prefix}mimic_robotiq_85_4">
+      <plugin filename="libroboticsgroup_gazebo_mimic_joint_plugin.so" name="${prefix}mimic_robotiq_85_4">
         <joint>${prefix}robotiq_85_left_knuckle_joint</joint>
         <mimicJoint>${prefix}robotiq_85_left_finger_tip_joint</mimicJoint>
@@ -34,5 +34,5 @@
         <offset>0.0</offset>
       </plugin>
-      <plugin filename="libgazebo_mimic_joint_plugin.so" name="${prefix}mimic_robotiq_85_5">
+      <plugin filename="libroboticsgroup_gazebo_mimic_joint_plugin.so" name="${prefix}mimic_robotiq_85_5"> <!--libgazebo_mimic_joint_plugin-->
         <joint>${prefix}robotiq_85_left_knuckle_joint</joint>
         <mimicJoint>${prefix}robotiq_85_right_finger_tip_joint</mimicJoint>

File: ur_description/urdf/eefold.xacro (robot description, xacro)
@@ -5,4 +5,8 @@
         <origin xyz="0 0 0" rpy="0 0 0" />
     </xacro:robotiq_gripper>
+    <!--xacro:include filename="$(find robotiq_description)/urdf/robotiq_85_gripper.urdf.xacro" />
+    <xacro:robotiq_85_gripper prefix="" parent="tool0" >
+        <origin xyz="0 0 0" rpy="0 -1.507 3.14" />
+    </xacro:robotiq_85_gripper-->
     <!-- Equivalent to the OpenRAVE manipulator denso_robotiq_85_gripper -->
     <link name="ee_link" />

File: ur_description/urdf/robotiq_2f_85_macro.urdf.xacro (robot description, xacro)
@@ -259,5 +259,5 @@
             <axis xyz="0 -1 0" />
             <origin xyz="-0.0127 0.0 0.06142" rpy="0 0 0" />
-            <!--mimic joint="${prefix}robotiq_85_left_knuckle_joint" multiplier="-1" /-->
+            <mimic joint="${prefix}robotiq_85_left_knuckle_joint" multiplier="-1" />
         </joint>
         <joint name="${prefix}robotiq_85_left_finger_tip_joint" type="continuous">
@@ -266,5 +266,5 @@
             <axis xyz="0 -1 0" />
             <origin xyz="0.00563134 0.0 0.04718515" rpy="0 0 0" />
-            <!--mimic joint="${prefix}robotiq_85_left_knuckle_joint" multiplier="-1" /-->
+            <mimic joint="${prefix}robotiq_85_left_knuckle_joint" multiplier="-1" />
         </joint>
         <joint name="${prefix}robotiq_85_right_finger_tip_joint" type="continuous">
@@ -275,16 +275,4 @@
             <mimic joint="${prefix}robotiq_85_left_knuckle_joint" />
         </joint>
-        <!--joint name="${prefix}robotiq_85_left_inner_knuckle_tip_joint" type="continuous">
-            <parent link="${prefix}robotiq_85_left_finger_tip_link" />
-            <child link="${prefix}robotiq_85_left_inner_knuckle_link" />
-            <axis xyz="0 -1 0" />
-            <origin xyz="0 0 0" rpy="0 0 0" />
-        </joint>
-        <joint name="${prefix}robotiq_85_right_inner_knuckle_tip_joint" type="continuous">
-            <parent link="${prefix}robotiq_85_right_finger_tip_link" />
-            <child link="${prefix}robotiq_85_right_inner_knuckle_link" />
-            <axis xyz="0 -1 0" />
-            <origin xyz="0 0 0" rpy="0 0 0" />
-        </joint-->
     </xacro:macro>
 </robot>
